File: battery.kicad_sch (KiCad schematic)
At the start: 52 parts, among them Q1 PSMN2R0-30YLDX, Q10 2N7002, Q2 PSMN2R0-30YLDX, Q8 2N7002, Q9 2N7002, U15 MAX17205G+, U6 S-8252AAG-M6T1U, U7 BQ29209DRB

Commit message: E0005 schematic: all four sheets captured for SPEC v1.0, ERC 0
- power: USB-C CC Rd + ADC sense, U_IN TPS259470A with 3-level ILM legs, BQ25887 charger,
  TPS56637 2S->5 V buck with soft power latch, V5 sense, TPS629210 3V3 from V5
- battery: BQ29209/OV2/MID divider removed (owner Q2)
- mcu: SPEC 7 pin map (GPIO4/6/7 ADC, GPIO36 PWR_HOLD, GPIO48 EXP_INT_N), 9 V ESD on PB_RAW
- ports: 5 V OVLO/UVLO dividers, SMF5.0A, 10 uF at each eFuse input
- lib: TPS56637 symbol + TI RPA0010A footprint; E0003 references kept for unchanged parts

Co-Authored-By: Claude Opus 5.5 <noreply@anthropic.com>
Parts:
- removed C27, C28, C29, C30, C34: 100nF, Capacitor_SMD:C_0402_1005Metric, symbol Device:C_Small
- removed D10, D9: BAT54W, Package_TO_SOT_SMD:SOT-323_SC-70, symbol Diode:BAT54W
- removed Q10, Q8, Q9: 2N7002, Package_TO_SOT_SMD:SOT-23, symbol Transistor_FET:2N7002
- removed R21: 160R, Resistor_SMD:R_0402_1005Metric, symbol Device:R_Small_US
- removed R22: 261R, Resistor_SMD:R_0402_1005Metric, symbol Device:R_Small_US
- removed R23, R24: 100R, Resistor_SMD:R_0402_1005Metric, symbol Device:R_Small_US
- removed R25, R26: 100k, Resistor_SMD:R_0402_1005Metric, symbol Device:R_Small_US
- removed R27: 1k, Resistor_SMD:R_0402_1005Metric, symbol Device:R_Small_US
- removed R33, R34: 1M 1%, Resistor_SMD:R_0402_1005Metric, symbol Device:R_Small_US
- removed U7: BQ29209DRB, Package_SON:VSON-8-1EP_3x3mm_P0.65mm_EP1.65x2.4mm, symbol E0005:BQ29209
Connections:
- no-connect marks 6 -> 4
Other:
- note added: "Cell OV ladder: VREG 4.20 V -> S-8252 4.30 V -> BQ25887 cell OVP ~4.37 V. No BQ29209 (owner Q2)."
- note added: "FUEL GAUGE MAX17205 (stack-only, board GND)"
- note added: "PROTECTION S-8252AAG + LOW-SIDE FETS, R_SENSE"
- note added: "R 470R + C 100nF per ABLIC Table 11; 2k on VM. BAT54W clamps: reverse-cell protection of VC."
- note added: "RT1 (NTC1) -> BQ25887 TS, RT2 (NTC2) -> gauge AIN1; both between the cells."
- note removed: "100k to VDD = balancing OFF; Q10 (BAL_EN = TCA9535 P07, 100k gate pull-down) enables it."
- note removed: "BALANCER + SECONDARY OV BQ29209 (OV 4.30 V)"
- note removed: "FUEL GAUGE MAX17205 (stack-only, board GND), MID ADC divider"
- note removed: "MID divider 1M/1M + 100 nF -> GPIO4 (coarse cell-1 voltage, board-GND referenced)."
- note removed: "OUT high on cell OV (4.30 V): Q8 -> charger HIZ (ILIM_HIZ low), Q9 -> OV2_N to TCA9535 P15."
- note removed: "PRIMARY PROTECTION S-8252AAG + LOW-SIDE FETS, R_SENSE"
- note removed: "R1/R2 470R + C 100nF per ABLIC Table 11; R3 2k on VM. BAT54W clamps: reverse-cell protection of VC."
- note removed: "RT1 -> charger TS, RT2 -> gauge AIN1; both between the cells."
- note removed: "Values per BQ29209 Fig. 9 (260R -> 261R E96). CD 0.1 uF -> ~0.9 s OV delay. CB_EN active-low (stack-referenced):"
- title: E0003 ESP32 control box mainboard -> E0005 ESP32-S3 5 V controller
