File: mcu.kicad_sch (KiCad schematic)
At the start: 54 parts, among them J10 FH12-18S-0.5SH, J12 SM02B-GHS-TB, J6 SM02B-GHS-TB, J7 SM02B-GHS-TB, J8 SM02B-GHS-TB, J9 SM02B-GHS-TB, SW1 PWR, SW2 BOOT, SW3 RESET, U1 ESP32-S3-WROOM-1-N16R2

Commit message: E0005 schematic: all four sheets captured for SPEC v1.0, ERC 0
- power: USB-C CC Rd + ADC sense, U_IN TPS259470A with 3-level ILM legs, BQ25887 charger,
  TPS56637 2S->5 V buck with soft power latch, V5 sense, TPS629210 3V3 from V5
- battery: BQ29209/OV2/MID divider removed (owner Q2)
- mcu: SPEC 7 pin map (GPIO4/6/7 ADC, GPIO36 PWR_HOLD, GPIO48 EXP_INT_N), 9 V ESD on PB_RAW
- ports: 5 V OVLO/UVLO dividers, SMF5.0A, 10 uF at each eFuse input
- lib: TPS56637 symbol + TI RPA0010A footprint; E0003 references kept for unchanged parts

Co-Authored-By: Claude Opus 5.5 <noreply@anthropic.com>
Parts:
- removed D12: PESD5V0L1UL, Diode_SMD:D_SOD-882, symbol Diode:PESD5V0L1UL
- removed R39: 10k, Resistor_SMD:R_0402_1005Metric, symbol Device:R_Small_US
- removed R61: 0R, Resistor_SMD:R_0402_1005Metric, symbol Device:R_Small_US
- added D12: TPD1E10B09, Diode_SMD:D_0402_1005Metric, symbol Device:D_TVS
Connections:
- net EXP_INT_N: now also U1.25 (IO48); no longer U1.7 (IO7)
- net GND: now also D12.2 (A2)
- net PB_RAW: now also D12.1 (A1)
- net SPARE37: now also R60.1
- net CHG_QON_N renamed PL_PULL
- net EYESPI_GP2: no longer names the net of J10.18 (Pin_18)
- net PD_ALERT_N renamed CC1_SENSE
- net SPARE36 renamed PWR_HOLD
- net PWR_HOLD: no longer R60.1
- net VMID_SENSE renamed V5_SENSE
- new net CC2_SENSE: U1.7 (IO7)
Other:
- note added: "ADC1: GPIO4 V5_SENSE, GPIO6/7 CC1/CC2_SENSE (power sheet). GPIO48 = TCA9535 INT."
- note added: "N16R2: quad PSRAM, GPIO35-37 usable (35 gauge ALRT, 36 PWR_HOLD, 37 spare)."
- note added: "POWER BUTTON SW1 + J12 (soft power latch on, GPIO21 sense)"
- note added: "Press: PB_RAW low -> PL_PULL low (latch on, power sheet) + GPIO21 low (wake). Long press: firmware"
- note added: "SCL/SDA = mux ch5 (4.7k on ports sheet). Unused selects 10k up. GP1 via DNP 0R from GPIO37; GP2 NC."
- note added: "drops PWR_HOLD. PB_RAW floats up to BAT+ when idle: 9 V ESD (not PESD5V0), GPIO21 diode blocks it."
- note removed: "N16R2: quad PSRAM, GPIO35-37 usable (35 = gauge ALRT, 36/37 spare)."
- note removed: "POWER BUTTON (ship mode on/off) SW1 + J12"
- note removed: "Press: BQ25798 QON low (exits ship mode) + GPIO21 low (wake). Long press -> firmware ship mode."
- note removed: "SCL/SDA = mux ch5 (4.7k on ports sheet). Unused selects 10k up. GP1/GP2 via DNP 0R from GPIO36/37."
- title: E0003 ESP32 control box mainboard -> E0005 ESP32-S3 5 V controller
