File: ports.kicad_sch (KiCad schematic)
At the start: 113 parts, among them J1 SM04B-GHS-TB, J2 SM04B-GHS-TB, J3 SM04B-GHS-TB, J4 SM04B-GHS-TB, J5 SM06B-GHS-TB, Q3 2N7002, Q4 2N7002, Q5 2N7002, Q6 2N7002, Q7 2N7002, U10 TPS259470ARPW, U11 TPS259470ARPW, U12 TPS259470ARPW, U13 TPS259470ARPW, U14 TPS259470ARPW, U8 PCA9548APW, U9 TCA9535PWR

Commit message: E0005 schematic: all four sheets captured for SPEC v1.0, ERC 0
- power: USB-C CC Rd + ADC sense, U_IN TPS259470A with 3-level ILM legs, BQ25887 charger,
  TPS56637 2S->5 V buck with soft power latch, V5 sense, TPS629210 3V3 from V5
- battery: BQ29209/OV2/MID divider removed (owner Q2)
- mcu: SPEC 7 pin map (GPIO4/6/7 ADC, GPIO36 PWR_HOLD, GPIO48 EXP_INT_N), 9 V ESD on PB_RAW
- ports: 5 V OVLO/UVLO dividers, SMF5.0A, 10 uF at each eFuse input
- lib: TPS56637 symbol + TI RPA0010A footprint; E0003 references kept for unchanged parts

Co-Authored-By: Claude Opus 5.5 <noreply@anthropic.com>
Parts:
- removed D19, D21, D23, D25, D27: SMF9.0A, Diode_SMD:D_SOD-123F, symbol Diode:SMF9V0A
- removed R91: 10k, Resistor_SMD:R_0402_1005Metric, symbol Device:R_Small_US
- added D19, D21, D23, D25, D27: SMF5.0A, Diode_SMD:D_SOD-123F, symbol Diode:SMF5V0A
- C48, C51, C54, C57, C60: value 100nF -> 10uF; footprint Capacitor_SMD:C_0402_1005Metric -> Capacitor_SMD:C_0805_2012Metric; MPN GRM155R71H104KE14D -> TMK212BBJ106MG-T; Manufacturer Murata Electronics -> Taiyo Yuden; Supplier PN 490-10700-1-ND -> 587-6025-1-ND; Voltage 50V -> 25V
- R102, R109, R116, R123, R95: value 232k 1% -> 365k 1%; MPN RC0402FR-07232KL -> RC0402FR-07365KL; Supplier PN YAG3062CT-ND -> YAG3133CT-ND
- R104, R111, R118, R125, R97: value 137k 1% -> 249k 1%; MPN RC0402FR-07137KL -> RC0402FR-07249KL; Supplier PN YAG2972CT-ND -> 311-249KLRCT-ND
Connections:
- net GND: now also D19.2 (A2), D21.2 (A2), D23.2 (A2), D25.2 (A2), D27.2 (A2)
- net BAL_EN renamed USB_ILIM_3A0
- net CHG_CE_N renamed CHG_CD
- net EXP_P06 renamed USB_ILIM_1A5
- net EXP_P16 renamed CHG_PG_N
- net EXP_P17 renamed BUCK_PG
- net OV2_N renamed USBIN_FLT_N
- net PBUS_1 renamed V5_1
- net V5_1: now also D19.1 (A1)
- net PBUS_2 renamed V5_2
- net V5_2: now also D21.1 (A1)
- net PBUS_3 renamed V5_3
- net V5_3: now also D23.1 (A1)
- net PBUS_4 renamed V5_4
- net V5_4: now also D25.1 (A1)
- net PBUS_5 renamed V5_5
- net V5_5: now also D27.1 (A1)
- net VSYS renamed V5
Other:
- note added: "(+4 at the buck output)."
- note added: "-> charging OFF; P06/P07 USB_ILIM_1A5/3A0 100k down at the leg FETs -> U_IN 0.50 A."
- note added: "2 x 47 uF/16 V on V5"
- note added: "I_LIM 0.87 A (0.74-1.00); OVLO 6.02/5.47 V; UVLO 4.49/4.08 V"
- note added: "I_LIM 2.03 A (1.80-2.20); OVLO 6.02/5.47 V; UVLO 4.49/4.08 V"
- note added: "P10-P14 port FLT, P15 USBIN_FLT_N, P16 CHG_PG_N, P17 BUCK_PG: inputs, 10k pull-ups. INT -> GPIO48."
- note added: "PORT 1: J1 5V GH4 E0001, 0.87 A"
- note added: "PORT 2: J2 5V GH4 E0001, 0.87 A"
- note added: "PORT 3: J3 5V GH4 E0001, 0.87 A"
- note added: "PORT 4: J4 5V GH4 E0001, 0.87 A"
- note added: "PORT 5: J5 5V GH6 E0002, 2.0 A"
- note added: "Reset state (all inputs): P00-P04 PORTn_OFF 100k up -> ports OFF; P05 CHG_CD 10k up (power sheet)"
- note added: "Silkscreen: "5V" + "1" + "E0001""
- note added: "Silkscreen: "5V" + "2" + "E0001""
- note added: "Silkscreen: "5V" + "3" + "E0001""
- note added: "Silkscreen: "5V" + "4" + "E0001""
- note added: "Silkscreen: "5V" + "5" + "E0002""
- note added: "V5 BULK"
- note added: "ch0-ch3 -> J1-J4 (E0001 5 V rev.), ch4 -> J5 (E0002 5 V rev.), ch5 -> EYESPI touch: 4.7k to 3V3."
- note added: "next to the eFuse group"
- note removed: "-> charging OFF; P07 BAL_EN pulled down at Q10 -> balancing OFF. P10-P15 inputs with 10k pull-ups."
- note removed: "2 x 47 uF/16 V on VSYS"
- note removed: "INT -> GPIO7. P06/P16/P17 spare (10k pull-ups)."
- note removed: "I_LIM 0.87 A (0.74-1.00); OVLO 9.96/9.05 V; UVLO 6.37/5.79 V"
- note removed: "I_LIM 2.03 A (1.80-2.20); OVLO 9.96/9.05 V; UVLO 6.37/5.79 V"
- note removed: "PBUS BULK"
- note removed: "PORT 1: J1 GH4 E0001 rev C, 0.87 A"
- note removed: "PORT 2: J2 GH4 E0001 rev C, 0.87 A"
- note removed: "PORT 3: J3 GH4 E0001 rev C, 0.87 A"
- note removed: "PORT 4: J4 GH4 E0001 rev C, 0.87 A"
- note removed: "PORT 5: J5 GH6 E0002 rev B, 2.0 A"
- note removed: "Reset state (all inputs): P00-P04 PORTn_OFF 100k up -> ports OFF; P05 CHG_CE_N 10k up (charger sheet)"
- note removed: "Silkscreen: "PBUS 6-9 V" + "1" + "E0001""
- note removed: "Silkscreen: "PBUS 6-9 V" + "2" + "E0001""
- note removed: "Silkscreen: "PBUS 6-9 V" + "3" + "E0001""
- note removed: "Silkscreen: "PBUS 6-9 V" + "4" + "E0001""
- note removed: "Silkscreen: "PBUS 6-9 V" + "5" + "E0002""
- note removed: "ch0-ch3 -> J1-J4 (E0001 rev C), ch4 -> J5 (E0002 rev B), ch5 -> EYESPI touch: 4.7k to 3V3."
- note removed: "next to the eFuse group."
- title: E0003 ESP32 control box mainboard -> E0005 ESP32-S3 5 V controller

Commit message: E0005 schematic for SPEC v1.1: TPS56637 L1 3.3 uH IHLP3232 + V5 bulk 2 x 47 uF (~88 uF eff.), port UVLO 1M/402k, USB-only back-feed analysis, ERC 0
- remove C61/C62 and the v1.0 extra buck caps (C77/C78 left unused); V5 effective-C table from Samsung DC-bias data
- port EN/UVLO 402k on all 5 ports (4.19/3.80 V), TPS629210 dropout check at 3.8 V
- O-1 closed, O-2 closed as SPEC v1.1 8.5/13; new section: V5 -> BAT+ back-feed with no battery (a)-(e)
- BOM regenerated; placement notes updated for the 8.6 x 8.2 mm inductor

Co-Authored-By: Claude Opus 5.5 <noreply@anthropic.com>
Parts:
- removed C61, C62: 47uF, Capacitor_SMD:C_1210_3225Metric, symbol Device:C_Small
- R102, R109, R116, R123, R95: value 365k 1% -> 402k 1%; MPN RC0402FR-07365KL -> RC0402FR-07402KL; Supplier PN YAG3133CT-ND -> YAG3151CT-ND
Other:
- note added: "I_LIM 0.87 A (0.74-1.00); OVLO 6.02/5.47 V; UVLO 4.19/3.80 V"
- note added: "I_LIM 2.03 A (1.80-2.20); OVLO 6.02/5.47 V; UVLO 4.19/3.80 V"
- note removed: "(+4 at the buck output)."
- note removed: "2 x 47 uF/16 V on V5"
- note removed: "I_LIM 0.87 A (0.74-1.00); OVLO 6.02/5.47 V; UVLO 4.49/4.08 V"
- note removed: "I_LIM 2.03 A (1.80-2.20); OVLO 6.02/5.47 V; UVLO 4.49/4.08 V"
- note removed: "V5 BULK"
- note removed: "next to the eFuse group"
