File: power.kicad_sch (KiCad schematic)
At the start: 47 parts, among them J11 USB4105-GF-A, U2 BQ25798RQMR, U3 STUSB4500QTR, U4 USBLC6-2SC6, U5 TPS629210DRL

Commit message: E0005 schematic: all four sheets captured for SPEC v1.0, ERC 0
- power: USB-C CC Rd + ADC sense, U_IN TPS259470A with 3-level ILM legs, BQ25887 charger,
  TPS56637 2S->5 V buck with soft power latch, V5 sense, TPS629210 3V3 from V5
- battery: BQ29209/OV2/MID divider removed (owner Q2)
- mcu: SPEC 7 pin map (GPIO4/6/7 ADC, GPIO36 PWR_HOLD, GPIO48 EXP_INT_N), 9 V ESD on PB_RAW
- ports: 5 V OVLO/UVLO dividers, SMF5.0A, 10 uF at each eFuse input
- lib: TPS56637 symbol + TI RPA0010A footprint; E0003 references kept for unchanged parts

Co-Authored-By: Claude Opus 5.5 <noreply@anthropic.com>
Parts:
- removed C10, C13, C14, C15, C16, C17, C19, C5, C6: 10uF, Capacitor_SMD:C_0805_2012Metric, symbol Device:C_Small
- removed C12: 47nF, Capacitor_SMD:C_0402_1005Metric, symbol Device:C_Small
- removed C21: 1nF, Capacitor_SMD:C_0402_1005Metric, symbol Device:C_Small
- removed C3, C4: 1uF, Capacitor_SMD:C_0402_1005Metric, symbol Device:C_Small
- removed C7: 100nF, Capacitor_SMD:C_0402_1005Metric, symbol Device:C_Small
- removed D1: TVS2200DRVR, Package_SON:WSON-6-1EP_2x2mm_P0.65mm_EP1x1.6mm, symbol Power_Protection:TVS2200DRV
- removed R4: 100k, Resistor_SMD:R_0402_1005Metric, symbol Device:R_Small_US
- removed R5: 1k, Resistor_SMD:R_0402_1005Metric, symbol Device:R_Small_US
- removed R6: 100R, Resistor_SMD:R_0402_1005Metric, symbol Device:R_Small_US
- removed R7: 8.2k 1%, Resistor_SMD:R_0402_1005Metric, symbol Device:R_Small_US
- removed R8: 10k 1%, Resistor_SMD:R_0402_1005Metric, symbol Device:R_Small_US
- removed R9: 21.5k 1%, Resistor_SMD:R_0402_1005Metric, symbol Device:R_Small_US
- removed U2: BQ25798RQMR, Package_DFN_QFN:Texas_RQM0029A_VQFN-29_4x4mm_P0.4mm, symbol Battery_Management:BQ25798
- removed U3: STUSB4500QTR, Package_DFN_QFN:QFN-24-1EP_4x4mm_P0.5mm_EP2.7x2.7mm, symbol Interface_USB:STUSB4500QTR
- added C63, C64: 1nF, Capacitor_SMD:C_0402_1005Metric, symbol Device:C_Small
- added C65, C68, C73, C74: 100nF, Capacitor_SMD:C_0402_1005Metric, symbol Device:C_Small
- added C66: 1.8nF, Capacitor_SMD:C_0402_1005Metric, symbol Device:C_Small
- added C67: 22nF, Capacitor_SMD:C_0402_1005Metric, symbol Device:C_Small
- added C69, C70, C75, C76, C77, C78: 47uF, Capacitor_SMD:C_1210_3225Metric, symbol Device:C_Small
- added C71, C72: 10uF, Capacitor_SMD:C_0805_2012Metric, symbol Device:C_Small
- added C79: 100pF, Capacitor_SMD:C_0402_1005Metric, symbol Device:C_Small
- added D1: SMF9.0A, Diode_SMD:D_SOD-123F, symbol Diode:SMF9V0A
- added L2: 1uH, Inductor_SMD:L_Vishay_IHLP-2525, symbol Device:L
- added Q11, Q12, Q14: 2N7002, Package_TO_SOT_SMD:SOT-23, symbol Transistor_FET:2N7002
- added Q13: AO3401A, Package_TO_SOT_SMD:SOT-23, symbol Transistor_FET:AO3401A
- added R129, R130: 5.1k 1%, Resistor_SMD:R_0402_1005Metric, symbol Device:R_Small_US
- added R131, R132, R144, R149: 10k, Resistor_SMD:R_0402_1005Metric, symbol Device:R_Small_US
- added R133, R135: 1M 1%, Resistor_SMD:R_0402_1005Metric, symbol Device:R_Small_US
- added R134: 390k 1%, Resistor_SMD:R_0402_1005Metric, symbol Device:R_Small_US
- added R136: 249k 1%, Resistor_SMD:R_0402_1005Metric, symbol Device:R_Small_US
- added R137: 6.65k 1%, Resistor_SMD:R_0402_1005Metric, symbol Device:R_Small_US
- added R138: 3.83k 1%, Resistor_SMD:R_0402_1005Metric, symbol Device:R_Small_US
- added R139, R141, R142, R143, R150: 100k, Resistor_SMD:R_0402_1005Metric, symbol Device:R_Small_US
- added R140: 2.32k 1%, Resistor_SMD:R_0402_1005Metric, symbol Device:R_Small_US
- added R145: 374R 1%, Resistor_SMD:R_0402_1005Metric, symbol Device:R_Small_US
- added R146: 300R, Resistor_SMD:R_0402_1005Metric, symbol Device:R_Small_US
- added R147: 39R 1% 1W, Resistor_SMD:R_2512_6332Metric, symbol Device:R_Small_US
- added R148: 39k, Resistor_SMD:R_0402_1005Metric, symbol Device:R_Small_US
- added R151: 200k 1%, Resistor_SMD:R_0402_1005Metric, symbol Device:R_Small_US
- added R152: 53.6k 1%, Resistor_SMD:R_0402_1005Metric, symbol Device:R_Small_US
- added R153: 69.8k 1%, Resistor_SMD:R_0402_1005Metric, symbol Device:R_Small_US
- added R154: 10k 1%, Resistor_SMD:R_0402_1005Metric, symbol Device:R_Small_US
- added R155: 20k, Resistor_SMD:R_0402_1005Metric, symbol Device:R_Small_US
- added U16: TPS259470ARPW, E0005:TI_RPW0010A_VQFN-HR-10_2x2mm_P0.475mm, symbol E0005:TPS259470L
- added U17: TPS56637RPAR, E0005:TI_RPA0010A_VQFN-HR-10_3x3mm, symbol E0005:TPS56637
- added U2: BQ25887RGET, Package_DFN_QFN:Texas_RGE0024H_VQFN-24-1EP_4x4mm_P0.5mm_EP2.7x2.7mm, symbol Battery_Management:BQ25887RGE
- C22: value 4.7uF -> 10uF; footprint Capacitor_SMD:C_0603_1608Metric -> Capacitor_SMD:C_0805_2012Metric; MPN GRM188R61E475KE11D -> TMK212BBJ106MG-T; Manufacturer Murata Electronics -> Taiyo Yuden; Supplier PN 490-7203-1-ND -> 587-6025-1-ND
Connections:
- net VSYS is gone; now on net V5: C22.1, C23.1, U5.6 (VIN), U5.7 (EN)
- net +3V3: now also R144.1
- net BAT+: now also C71.1, C72.1, C73.1, Q13.2 (S), R148.1, U17.8 (VIN), U2.13 (BAT), U2.14 (BAT)
- net BUCK_SW: now also L1.1, C74.2, U17.6 (SW); no longer L3.1, U5.4 (SW)
- net CC1: now also R129.1, R131.1
- net CC2: now also R130.1, R132.1
- net CHG_INT_N: now also U2.6 (~{INT})
- net CHG_STAT: now also U2.2 (STAT)
- net CHG_TS: now also U2.7 (TS)
- net GND: now also C63.2, C64.2, C65.2, C66.2, C67.2, C68.2, C69.2, C70.2, C71.2, C72.2, C73.2, C75.2, C76.2, C77.2, C78.2, D1.2 (A2), Q11.2 (S), Q12.2 (S), Q14.2 (S), R129.2, R130.2, R134.2, R136.2, R137.2, R139.2, R141.2, R143.2, R145.2, R150.2, R152.2, R154.2, U16.8 (GND), U17.10 (MODE), U17.3 (AGND), U17.9 (PGND), U2.19 (GND), U2.20 (GND), U2.25 (GND)
- net I2C0_SCL: now also U2.5 (SCL)
- net I2C0_SDA: now also U2.4 (SDA)
- net REGN: now also U2.11 (REGN)
- net VBUS: now also C65.1, D1.1 (A1), R133.1, R135.1, U16.5 (IN), U2.23 (VBUS)
- net CHG_BTST1 renamed CHG_BTST
- net CHG_BTST: now also U2.12 (BTST)
- net CHG_CE_N renamed CHG_CD
- net CHG_CD: now also U2.3 (CD)
- net CHG_SW1 renamed CHG_SW
- net CHG_SW: now also L2.2, U2.17 (SW), U2.18 (SW); no longer L1.1
- net CHG_SW2 renamed V5
- net V5: now also C75.1, C76.1, C77.1, C78.1, R142.1, R153.1, R155.1, U16.6 (OUT)
- net PMID renamed CHG_PMID
- net CHG_PMID: now also L2.1, U2.21 (PMID), U2.22 (PMID)
- new net: Q11.3 (D), R138.2
- new net: C79.1, R155.2
- new net: Q12.3 (D), R140.2
- new net: Q13.1 (G), R148.2, R149.1
- new net: Q13.3 (D), R151.1
- new net BUCK_BOOT: C74.1, U17.7 (BOOT)
- new net BUCK_EN: R151.2, R152.1, U17.1 (EN)
- new net BUCK_FB: C79.2, R153.2, R154.1, U17.2 (FB)
- new net BUCK_PG: U17.4 (PG)
- new net BUCK_SW_3V3: L3.1, U5.4 (SW)
- new net CC1_SENSE: C63.1, R131.2
- new net CC2_SENSE: C64.1, R132.2
- new net CHG_CBSET: R147.1, U2.10 (CBSET)
- new net CHG_ILIM: R145.1, U2.8 (ILIM)
- new net CHG_MID: R146.1, U2.9 (MID)
- new net CHG_PG_N: U2.1 (~{PG})
- new net CHG_PSEL: R144.2, U2.24 (PSEL)
- new net CHG_SNS: C69.1, C70.1, U2.15 (SNS), U2.16 (SNS)
- new net MID: R146.2, R147.2
- new net PL_PULL: Q14.3 (D), R149.2
- new net PWR_HOLD: Q14.1 (G), R150.1
- new net UIN_DVDT: C66.1, U16.7 (DVDT)
- new net UIN_EN: R133.2, R134.1, U16.1 (EN/UVLO)
- new net UIN_ILM: R137.1, R138.1, R140.1, U16.9 (ILM)
- new net UIN_ITIMER: C67.1, U16.10 (ITIMER)
- new net UIN_OVLO: R135.2, R136.1, U16.2 (OVLO)
- new net USBIN_FLT_N: U16.4 (~{FLT})
- new net USB_ILIM_1A5: Q11.1 (G), R139.1
- new net USB_ILIM_3A0: Q12.1 (G), R141.1
- new net V5_SENSE: C68.1, R142.2, R143.1
- no-connect marks 14 -> 6
Other:
- note added: "(MCU sheet) pulls PL_PULL -> Q_PL on -> buck on -> firmware sets PWR_HOLD (GPIO36). Off: PWR_HOLD low."
- note added: "(no reverse current: V5 diode-OR with U_IN). L1 2.2 uH, 4 x 47 uF here + 2 at the ports (SPEC 5.1.1)."
- note added: "10k + 1 nF to GPIO6/7 (ADC1): ~0.41 V default, ~0.92 V 1.5 A, ~1.68 V 3.0 A."
- note added: "3V3 BUCK TPS629210 (from V5, 1 A)"
- note added: "BAT 10 uF, REGN 4.7 uF. TS: REGN 5.23k / 30.1k || NTC1 103AT-2 (battery sheet) -> JEITA 0-60 C."
- note added: "BAT = BAT+ after F1. SNS is the boost output (internal R_SNS to BAT): caps only."
- note added: "BATTERY -> V5 BUCK TPS56637 (4.80 V, Eco-mode) + SOFT POWER LATCH"
- note added: "CD 10k up -> HIZ / charging OFF at reset (TCA9535 P05 drives low). PG -> P16, INT -> GPIO5."
- note added: "CHARGER BQ25887 (I2C0 0x6A): 5 V USB -> 2S boost, 1.5 MHz, balancing"
- note added: "D+/D- 90 ohm diff., 0R to GPIO20/19. CC: 5.1k Rd each (dead-battery safe);"
- note added: "D1 SMF9.0A: 15.4 V clamp < 20 V BQ25887 / TPS25947 abs max. USBLC6 VBUS pin to +3V3."
- note added: "EN 200k / 53.6k from Q_PL: 5.38 V rising (5.76 V max), 4.30 V falling (Ip 1 uA, Ih 4 uA); 1.99 V at 8.4 V."
- note added: "EN tied to V5; 100 % duty down to ~3.5 V V5. PG unused."
- note added: "FB 69.8k/10k: 0.6 x (1 + 6.98) = 4.79 V. FF 20k + 100 pF (Table 4, 5 V row). MODE = GND -> Eco-mode"
- note added: "ILIM 374R -> 2.97 A hardware cap (K_ILIM 1110). PSEL 10k up -> 500 mA default input limit."
- note added: "ITIMER 22 nF (~18 ms), dVdt 1.8 nF. FLT -> TCA9535 P15 (low = at its limit / TSD)."
- note added: "I_LIM = 3334 / R_ILM: 6.65k -> 0.50 A (reset), || 3.83k -> 1.37 A (P06), || 2.32k -> 2.81 A (P06+P07)."
- note added: "Latch: Q_PL AO3401A (-30 V, +-12 V), 39k gate-source -> VGS -6.7 V at 8.4 V. Press: PB_RAW low -> D13"
- note added: "Legs are cumulative: never P07 without P06. 100k gate pull-downs -> 0.50 A at reset."
- note added: "MID 300R (bottom-cell reverse protection), CBSET 39R 2512 -> ~108 mA balancing (0.45 W)."
- note added: "MODE/S-CONF 27.4k: VSET mode, auto PFM/PWM, output discharge. FB/VSET open -> 3.3 V."
- note added: "OVLO 1M/249k: 6.02 V rising. EN/UVLO 1M/390k: 4.28 V rising / 3.88 V falling."
- note added: "PG -> TCA9535 P17 (10k up on ports sheet)."
- note added: "Per BQ25887 Fig. 69: VBUS 1 uF, PMID 2 x 10 uF/25 V, L 1 uH PMID -> SW, BTST 47 nF, SNS 2 x 47 uF/16 V,"
- note added: "Thermal: keep the SPEC 5.6.1 copper (IN/OUT pours >= 80 mm2, 6 vias each, no reliefs)."
- note added: "USB + battery: keep PWR_HOLD high (EN low turns on the 200R SW discharge, ~25 mA from V5)."
- note added: "USB INPUT eFUSE U_IN TPS259470A: VBUS -> V5, 0.50 / 1.37 / 2.81 A"
- note added: "USB-C J11 (5 V, no PD), VBUS TVS, USB ESD, CC Rd + sense"
- note added: "V5 / 2 -> GPIO4 (ADC1_CH3), 2.75 V at 5.5 V."
- note added: "V5 SENSE (GPIO4), POWER FLAGS"
- note added: "V5 and BAT+ are driven by U16 OUT / U2 BAT."
- note removed: "3V3 BUCK TPS629210 (from VSYS, 1 A)"
- note removed: "ADDR0/1 = GND -> 0x28. RESET 100k to GND. VSYS = GND (powered from VBUS only)."
- note removed: "BQ29209 OV2 FET (battery sheet) pulls ILIM_HIZ < 0.75 V -> HIZ."
- note removed: "CE: 10k pull-up -> charging OFF at reset; TCA9535 P05 enables. QON <- power button."
- note removed: "CHARGER / POWER PATH BQ25798 (I2C0 0x6B), 2S, 750 kHz"
- note removed: "D+/D- 90 ohm diff., 0R footprints to GPIO20/19."
- note removed: "D+/D- not used (IINDPM set by firmware from the STUSB4500 contract). SDRV: 1 nF (no ship FET)."
- note removed: "FB/VSET open (>= 249k) -> 3.3 V. EN tied to VSYS. PG unused."
- note removed: "MODE/S-CONF 27.4k: VSET mode, auto PFM/PWM, output discharge."
- note removed: "NVM (write once): PDO1 5 V, PDO2 9 V >= 2 A, PDO3 15 V >= 2 A, REQ_SRC_CURRENT = 1."
- note removed: "Open-drain flags ATTACH/POWER_OKx/GPIO/A_B_SIDE/VBUS_EN_SNK and DISCH unused."
- note removed: "PROG 8.2k: 2S, 750 kHz. ILIM_HIZ = 5 V x 21.5/31.5 = 3.41 V -> IINDPM clamp 3.0 A;"
- note removed: "TS: REGN 5.23k / 30.1k || NTC1 (103AT-2, battery sheet) -> JEITA 0-60 C."
- note removed: "USB-C J11, VBUS TVS, USB ESD"
- note removed: "USB-PD SINK STUSB4500 (I2C0 0x28), PDO 15 V / 9 V / 5 V"
- note removed: "USBLC6 VBUS pin to +3V3 (VBUS reaches 15 V)."
- note removed: "VAC1 = VAC2 = VBUS, ACDRV1/2 = GND: single input, no ACFET (datasheet Table 7-5)."
- title: E0003 ESP32 control box mainboard -> E0005 ESP32-S3 5 V controller

Commit message: E0005 schematic for SPEC v1.1: TPS56637 L1 3.3 uH IHLP3232 + V5 bulk 2 x 47 uF (~88 uF eff.), port UVLO 1M/402k, USB-only back-feed analysis, ERC 0
- remove C61/C62 and the v1.0 extra buck caps (C77/C78 left unused); V5 effective-C table from Samsung DC-bias data
- port EN/UVLO 402k on all 5 ports (4.19/3.80 V), TPS629210 dropout check at 3.8 V
- O-1 closed, O-2 closed as SPEC v1.1 8.5/13; new section: V5 -> BAT+ back-feed with no battery (a)-(e)
- BOM regenerated; placement notes updated for the 8.6 x 8.2 mm inductor

Co-Authored-By: Claude Opus 5.5 <noreply@anthropic.com>
Parts:
- removed C77, C78: 47uF, Capacitor_SMD:C_1210_3225Metric, symbol Device:C_Small
- L1: value 2.2uH -> 3.3uH; footprint Inductor_SMD:L_Bourns_SRP7028A_7.3x6.6mm -> Inductor_SMD:L_Vishay_IHLP-3232; MPN SRP7028A-2R2M -> IHLP3232DZER3R3M11; Manufacturer Bourns Inc. -> Vishay Dale; Supplier PN SRP7028A-2R2MCT-ND -> 541-1352-1-ND
Other:
- note added: "(no reverse current). Table 4 5 V row: L1 3.3 uH; V5 total ~88 uF effective (2 x 47 uF + 6 x 10 uF), <= 100 uF."
- note removed: "(no reverse current: V5 diode-OR with U_IN). L1 2.2 uH, 4 x 47 uF here + 2 at the ports (SPEC 5.1.1)."
- moved on the sheet: C74

Commit message: E0005: U2 BQ25887RGET -> BQ25887RGER cut tape (296-53517-1-ND), BOM regenerated, ERC 0
Co-Authored-By: Claude Opus 5.5 <noreply@anthropic.com>
Parts:
- U2: value BQ25887RGET -> BQ25887RGER; MPN BQ25887RGET -> BQ25887RGER; Supplier PN 296-53518-2-ND -> 296-53517-1-ND
Changed lines of the file:
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@@
 			)
 		)
-		(property "Value" "BQ25887RGET"
+		(property "Value" "BQ25887RGER"
 			(at 119.38 220.98 0)
 			(effects
@@
 			)
 		)
-		(property "MPN" "BQ25887RGET"
+		(property "MPN" "BQ25887RGER"
 			(at 127 243.84 0)
 			(effects
@@
 			)
 		)
-		(property "Supplier PN" "296-53518-2-ND"
+		(property "Supplier PN" "296-53517-1-ND"
 			(at 127 243.84 0)
 			(effects
